File: nrf52/kicad/openrz67-nrf.kicad_pcb (KiCad board)
At the start: 2 copper layers, 29.5 x 29 mm, 14 parts, among them J1 Camera, J2 SWD, Q1 AO3401A, SW1 B3U-1000P, U1 E73-2G4M08S1F, U2 TLP172AM, U3 TLP172AM

Commit message: nrf52 pcb: 220 Ω relay drive, C3 at the module
Parts:
- added C3: 100nF, openrz67-nrf:C0402, F.Cu at (1.85, 18.4)
- R1, R2: value 330Ω -> 220Ω
- R3: value 330Ω -> 1kΩ
Routing:
- net GND: track 3.09 -> 4.65 mm
- net VDD: track 25.7 -> 26.7 mm
